File: OOS - optyczny odbiornik sygnalow/Sekcja_DCDC_Boost.kicad_sch (KiCad schematic)
At the start: 10 parts, among them U3 AP3015KTR-G1

Commit message: Add review notes for DCDC_Boost page
Changed lines of the file:
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@@
+		)
+	)
+	(text_box "Review notes:\n- Adding test points for circuits\n- Adding LED diodes for input and output\n- Changing U3 for IC with max output voltage +32V\n- Change output capacitor voltage rating more than 50V when output will be +32V\n- Remove 4 points cross connection for nets\n- Add net tie for SHDN pin, easy for test\n- Add pi filter ion the input\n- Change diode D4 due to the low breakdown voltage, Vout = 32V do not have enough margin\n- Add output solder jumper or 0R resistor, to measure only BOOST converter easier\n- Check the inductor on tdk.com current\n- R15, Voltage rating 75V, from where?\n- Change placement of pin 2 and 3 for U3 for better connection"
+		(exclude_from_sim no)
+		(at 93.98 151.13 0)
+		(size 59.055 46.355)
+		(margins 0.9525 0.9525 0.9525 0.9525)
+		(stroke
+			(width 0.2032)
+			(type solid)
+			(color 0 0 0 1)
+		)
+		(fill
+			(type color)
+			(color 255 68 62 1)
+		)
+		(effects
+			(font
+				(size 1.27 1.27)
+				(thickness 0.254)
+				(bold yes)
+			)
+			(justify left top)
 		)
 	)
@@
 		(on_board yes)
 		(dnp no)
-		(property "Reference" "R?"
+		(property "Reference" "R12"
 			(at 169.418 87.376 0)
 			(effects
@@
 		(on_board yes)
 		(dnp no)
-		(property "Reference" "U?"
+		(property "Reference" "U3"
 			(at 129.032 87.376 0)
 			(effects
@@
 		(on_board yes)
 		(dnp no)
-		(property "Reference" "#PWR?"
+		(property "Reference" "#PWR028"
 			(at 187.96 81.28 0)
 			(effects
@@
 		(on_board yes)
 		(dnp no)
-		(property "Reference" "C?"
+		(property "Reference" "C13"
 			(at 99.06 93.98 0)
 			(effects
@@
 		(on_board yes)
 		(dnp yes)
-		(property "Reference" "C?"
+		(property "Reference" "C14"
 			(at 179.07 87.63 0)
 			(effects
@@
 		(on_board yes)
 		(dnp no)
-		(property "Reference" "R?"
+		(property "Reference" "R13"
 			(at 98.298 81.28 0)
 			(effects
@@
 		(on_board yes)
 		(dnp no)
-		(property "Reference" "R?"
+		(property "Reference" "R15"
 			(at 169.418 105.156 0)
 			(effects
@@
 		(dnp no)
 		(fields_autoplaced yes)
-		(property "Reference" "#PWR?"
+		(property "Reference" "#PWR026"
 			(at 143.51 120.65 0)
 			(effects
@@
 		(on_board yes)
 		(dnp no)
-		(property "Reference" "D?"
+		(property "Reference" "D4"
 			(at 155.702 78.232 0)
 			(effects
@@
 		(on_board yes)
 		(dnp no)
-		(property "Reference" "#PWR?"
+		(property "Reference" "#PWR024"
 			(at 96.52 81.28 0)
 			(effects
@@
 		(on_board yes)
 		(dnp no)
-		(property "Reference" "C?"
+		(property "Reference" "C15"
 			(at 190.5 87.63 0)
 			(effects
@@
 		(dnp no)
 		(fields_autoplaced yes)
-		(property "Reference" "#PWR?"
+		(property "Reference" "#PWR027"
 			(at 187.96 120.65 0)
 			(effects
@@
 		(on_board yes)
 		(dnp no)
-		(property "Reference" "L?"
+		(property "Reference" "L1"
 			(at 131.064 78.994 90)
 			(effects
@@
 		(dnp no)
 		(fields_autoplaced yes)
-		(property "Reference" "#PWR?"
+		(property "Reference" "#PWR023"
 			(at 167.64 120.65 0)
 			(effects
@@
 		(dnp no)
 		(fields_autoplaced yes)
-		(property "Reference" "#PWR?"
+		(property "Reference" "#PWR025"
 			(at 96.52 111.76 0)
 			(effects
@@
 		(on_board yes)
 		(dnp yes)
-		(property "Reference" "C?"
+		(property "Reference" "C16"
 			(at 109.22 93.98 0)
 			(effects
